Commit message: Updated_2

File: mybot_description/urdf/mybot.xacro (robot description, xacro)
@@ -2,10 +2,11 @@
 <robot name="mybot" xmlns:xacro="http://www.ros.org/wiki/xacro">
 <!-- ++++++++++++++++++++++++++++++++ include xacro files +++++++++++++++++++++++++++++++ -->
-<!-- <xacro:include filename="$(find mybot_description)/urdf/mybot.gazebo"/> -->
+<!--<xacro:include filename="$(find mybot_description)/urdf/mybot.gazebo"/> -->
 <xacro:include filename="mybot_macros.xacro" />
 <xacro:include filename="mybot_material.xacro" />
-<xacro:include filename="mybot_base.xacro" />
+<xacro:include filename="gamed.xacro" />
+<!--<xacro:include filename="mybot_base.xacro" />
 <xacro:include filename="mybot_wheels.xacro" />
 <xacro:include filename="mybot_lidar.xacro" />
-<xacro:include filename="mybot_Pillars.xacro" />
+<xacro:include filename="mybot_Pillars.xacro" /> -->
 </robot>

File: mybot_description/urdf/mybot_base.xacro (robot description, xacro)
@@ -8,5 +8,5 @@
   <xacro:property name="wheel_distance" value="0.305"/>
   <xacro:property name="lidar_height" value="0.83"/>
-  <xacro:property name="imu_height" value="0.4025"/>
+  <xacro:property name="imu_height" value="0.001"/>
   <xacro:property name="caster_radius" value="0.0325"/>
   <xacro:property name="caster_distance" value="0.1525025"/>

File: mybot_description/urdf/mybot_lidar.xacro (robot description, xacro)
@@ -5,5 +5,5 @@
     <visual>
       <geometry>
-        <box size="0.03 0.03 0.01"/>
+        <box size="0.03 0.03 0.001"/>
       </geometry>
       <material name="green"><color rgba="0 1 0 1"/></material>
@@ -25,5 +25,5 @@
   </visual>
   <collision>
-    <origin xyz="0 0 0.45" rpy="0 0 0"/>
+    <origin xyz="0 0 0" rpy="0 0 0"/>
     <geometry>
       <mesh filename="package://mybot_description/meshes/RpLidar.stl" scale="0.001 0.001 0.001"/>
